File: hardware/schematic/CyberTrack.kicad_sch (KiCad schematic)
At the start: 13 parts, among them SW1 MASTER REQUEST / CONTACTS TBD, SW2 ACTUATOR ISOLATOR / TBD, U2 PROTECTION / TBD, U3 MASTER POWER / TBD

Commit message: fix(schematic): add ultrasonic interface
Add controller 3V3, GPIO1 TRIG and GPIO2 ECHO on A2 sheet 6, and synchronize the current motor-side annotation and documentation.

Preserve A1 history and record fresh six-page exports, zero ERC violations, 112 connectivity checks and five regression tests.
Other:
- added sheet Ultrasonic 3V3 interface (ultrasonic.kicad_sch)
- note added: "A2 design candidate. Protection / switching blocks are NOT implemented circuits."
- note removed: "A1 design candidate. Protection / switching blocks are NOT implemented circuits."
Changed lines of the file:
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@@
-(kicad_sch (version 20250114) (generator "cybertrack_schematic") (paper "A3") (title_block (title "CyberTrack / Power and isolation") (date "2026-10-26") (rev "A1") (company "CyberTrack") (comment 1 "MODULE INTERCONNECTION SCHEMATIC - NOT FOR FABRICATION") (comment 2 "Retain existing ESP32-S3 board; TBD items are unresolved") (comment 3 "Pin IDs identify signals, NOT physical header positions"))
+(kicad_sch (version 20250114) (generator "cybertrack_schematic") (paper "A3") (title_block (title "CyberTrack / Power and isolation") (date "2026-10-30") (rev "A2") (company "CyberTrack") (comment 1 "MODULE INTERCONNECTION SCHEMATIC - NOT FOR FABRICATION") (comment 2 "Retain existing ESP32-S3 board; TBD items are unresolved") (comment 3 "Pin IDs identify signals, NOT physical header positions"))
 (text "01  POWER INPUT AND DISTRIBUTION" (at 20.32 17.78 0) (effects (font (size 2.286 2.286)) (justify left top)))
-(text "A1 design candidate. Protection / switching blocks are NOT implemented circuits." (at 20.32 27.94 0) (effects (font (size 1.651 1.651)) (justify left top)))
+(text "A2 design candidate. Protection / switching blocks are NOT implemented circuits." (at 20.32 27.94 0) (effects (font (size 1.651 1.651)) (justify left top)))
 (symbol (lib_id "CyberTrack:Battery5V") (at 43.18 63.5 0) (unit 1) (in_bom no) (on_board no) (dnp no)(property "Reference" "BT1" (at 43.18 33.02 0) (effects (font (size 1.651 1.651))))
 (property "Value" "CK18650-1234S-NP / 5 V" (at 43.18 39.37 0) (effects (font (size 1.524 1.524))))
@@
 (sheet (at 88.9 254) (size 63.5 12.7) (stroke (width 0.254) (type default)) (fill (color 0 0 0 0)) (property "Sheetname" "Motor drive" (at 88.9 251.46 0) (effects (font (size 1.27 1.27)) (justify left bottom))) (property "Sheetfile" "drive.kicad_sch" (at 88.9 269.24 0) (effects (font (size 1.143 1.143)) (justify left top))) (instances (project "CyberTrack" (path "/5724a998-1735-5701-ac0a-8a8a7029fc41" (page "3")))))
 (sheet (at 157.48 254) (size 63.5 12.7) (stroke (width 0.254) (type default)) (fill (color 0 0 0 0)) (property "Sheetname" "Water and bubbles" (at 157.48 251.46 0) (effects (font (size 1.27 1.27)) (justify left bottom))) (property "Sheetfile" "effects.kicad_sch" (at 157.48 269.24 0) (effects (font (size 1.143 1.143)) (justify left top))) (instances (project "CyberTrack" (path "/5724a998-1735-5701-ac0a-8a8a7029fc41" (page "4")))))
-(sheet (at 226.06 254) (size 63.5 12.7) (stroke (width 0.254) (type default)) (fill (color 0 0 0 0)) (property "Sheetname" "Reserved ignition LV" (at 226.06 251.46 0) (effects (font (size 1.27 1.27)) (justify left bottom))) (property "Sheetfile" "ignition-lv.kicad_sch" (at 226.06 269.24 0) (effects (font (size 1.143 1.143)) (justify left top))) (instances (project "CyberTrack" (path "/5724a998-1735-5701-ac0a-8a8a7029fc41" (page "5")))))(sheet_instances (path "/" (page "1")))
+(sheet (at 226.06 254) (size 63.5 12.7) (stroke (width 0.254) (type default)) (fill (color 0 0 0 0)) (property "Sheetname" "Reserved ignition LV" (at 226.06 251.46 0) (effects (font (size 1.27 1.27)) (justify left bottom))) (property "Sheetfile" "ignition-lv.kicad_sch" (at 226.06 269.24 0) (effects (font (size 1.143 1.143)) (justify left top))) (instances (project "CyberTrack" (path "/5724a998-1735-5701-ac0a-8a8a7029fc41" (page "5")))))
+(sheet (at 20.32 231.14) (size 63.5 12.7) (stroke (width 0.254) (type default)) (fill (color 0 0 0 0)) (property "Sheetname" "Ultrasonic 3V3 interface" (at 20.32 228.6 0) (effects (font (size 1.27 1.27)) (justify left bottom))) (property "Sheetfile" "ultrasonic.kicad_sch" (at 20.32 246.38 0) (effects (font (size 1.143 1.143)) (justify left top))) (instances (project "CyberTrack" (path "/5724a998-1735-5701-ac0a-8a8a7029fc41" (page "6")))))(sheet_instances (path "/" (page "1")))
 )
