File: hardware/schematic/drive.kicad_sch (KiCad schematic)
At the start: 10 parts, among them M1 37R-520 / A, M2 37R-520 / B, U4 MT3608 / TARGET 12 V, U5 P13 / L298N

Commit message: fix(schematic): add ultrasonic interface
Add controller 3V3, GPIO1 TRIG and GPIO2 ECHO on A2 sheet 6, and synchronize the current motor-side annotation and documentation.

Preserve A1 history and record fresh six-page exports, zero ERC violations, 112 connectivity checks and five regression tests.
Other:
- note added: "Current firmware: A = right; B = left. Physical lead tracing / loaded tests still pending. Encoder conductors are not connected. Neither motor terminal is a fixed ground."
- note removed: "A = left candidate; B = right candidate. Vehicle direction still requires calibration. Encoder conductors are not connected. Neither motor terminal is a fixed ground."
Changed lines of the file:
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@@
-(kicad_sch (version 20250114) (generator "cybertrack_schematic") (paper "A3") (title_block (title "CyberTrack / Motor drive") (date "2026-10-26") (rev "A1") (company "CyberTrack") (comment 1 "MODULE INTERCONNECTION SCHEMATIC - NOT FOR FABRICATION") (comment 2 "Retain existing ESP32-S3 board; TBD items are unresolved") (comment 3 "Pin IDs identify signals, NOT physical header positions"))
+(kicad_sch (version 20250114) (generator "cybertrack_schematic") (paper "A3") (title_block (title "CyberTrack / Motor drive") (date "2026-10-30") (rev "A2") (company "CyberTrack") (comment 1 "MODULE INTERCONNECTION SCHEMATIC - NOT FOR FABRICATION") (comment 2 "Retain existing ESP32-S3 board; TBD items are unresolved") (comment 3 "Pin IDs identify signals, NOT physical header positions"))
 (text "03  EXTERNAL BOOST CONVERTER AND DUAL H-BRIDGE" (at 20.32 17.78 0) (effects (font (size 2.159 2.159)) (justify left top)))
 (symbol (lib_id "CyberTrack:MT3608") (at 78.74 83.82 0) (unit 1) (in_bom no) (on_board no) (dnp no)(property "Reference" "U4" (at 78.74 48.26 0) (effects (font (size 1.651 1.651))))
@@
 (wire (pts (xy 264.16 109.22) (xy 337.82 109.22)) (stroke (width 0) (type default)))
 (text "Remove ENA / ENB always-on jumpers.\nRetain only the verified regulator-jumper configuration.\nL298N +5V is intentionally unconnected.\n12 V bus is not guaranteed motor-terminal voltage." (at 20.32 121.92 0) (effects (font (size 1.651 1.651)) (justify left top)))
-(text "A = left candidate; B = right candidate.\nVehicle direction still requires calibration.\nEncoder conductors are not connected.\nNeither motor terminal is a fixed ground." (at 292.1 132.08 0) (effects (font (size 1.651 1.651)) (justify left top)))
+(text "Current firmware: A = right; B = left.\nPhysical lead tracing / loaded tests still pending.\nEncoder conductors are not connected.\nNeither motor terminal is a fixed ground." (at 292.1 132.08 0) (effects (font (size 1.651 1.651)) (justify left top)))
 (symbol (lib_id "CyberTrack:Pulldown") (at 53.34 203.2 0) (unit 1) (in_bom no) (on_board no) (dnp no)(property "Reference" "R1" (at 60.96 200.66 0) (effects (font (size 1.651 1.651)) (justify left)))
 (property "Value" "10k 1%" (at 60.96 207.01 0) (effects (font (size 1.524 1.524)) (justify left)))
